File: PowerConversionBoard.brd (EAGLE design)
At the start: 66 x 71.1 mm, 32 parts, among them U3 AZ1117EH-3.3TRG1

Commit message: playing with 3d models generated by eagle package
Parts:
- moved D1 0.14 mm to (30.8, 35.1), turned to 0 degrees
Connections:
- removed net N$1: U$1.3
- net FB: now also U$1.3
Routing:
- net FB: track 19.0 -> 22.0 mm
Changed lines of the file:
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@@
 </element>
 <element name="COUT" library="PowerComponents" package="CTAN(7.30_4.30MM)" value="100uF" x="62.723334375" y="26.605896875" smashed="yes"/>
-<element name="D1" library="Schottky Diode 8A - MBRD835LT4G" package="DPAK-3" value="SWITCHMODE_SCHOTTKY" x="30.7751625" y="35.00120625" smashed="yes" rot="R180">
-<attribute name="NAME" x="31.0751625" y="31.30120625" size="1.27" layer="25" rot="R180"/>
+<element name="D1" library="Schottky Diode 8A - MBRD835LT4G" package="DPAK-3" package3d_urn="urn:adsk.eagle:package:25915513/1" value="SWITCHMODE_SCHOTTKY" x="30.7944375" y="35.143434375" smashed="yes">
+<attribute name="NAME" x="30.4944375" y="38.843434375" size="1.27" layer="25"/>
 </element>
 <element name="RSEN" library="INA4181A4" package="CSS2H-2512" value="0.01" x="36.11173125" y="58.065553125" smashed="yes" rot="R90">
@@
 <contactref element="U3" pad="1"/>
 <via x="32.766" y="19.812" extent="1-16" drill="0.35"/>
-<wire x1="64.77" y1="55.626" x2="67.31" y2="55.626" width="0" layer="19" extent="1-1"/>
-<wire x1="57.277" y1="51.2826" x2="64.77" y2="55.626" width="0" layer="19" extent="1-1"/>
-<wire x1="57.2008" y1="60.1218" x2="64.77" y2="55.626" width="0" layer="19" extent="1-1"/>
-<wire x1="53.0962375" y1="66.551265625" x2="57.2008" y2="60.1218" width="0" layer="19" extent="1-1"/>
-<wire x1="45.466" y1="66.294" x2="53.0962375" y2="66.551265625" width="0" layer="19" extent="1-1"/>
-<wire x1="44.5262" y1="59.563" x2="45.466" y2="66.294" width="0" layer="19" extent="1-1"/>
-<wire x1="43.8658" y1="51.2826" x2="44.5262" y2="59.563" width="0" layer="19" extent="1-1"/>
-<wire x1="34.798" y1="66.548" x2="45.466" y2="66.294" width="0" layer="19" extent="1-1"/>
-<wire x1="67.244790625" y1="34.34263125" x2="57.277" y2="51.2826" width="0" layer="19" extent="1-1"/>
-<wire x1="65.943334375" y1="26.605896875" x2="67.244790625" y2="34.34263125" width="0" layer="19" extent="1-1"/>
-<wire x1="67.31" y1="8.636" x2="65.943334375" y2="26.605896875" width="0" layer="19" extent="1-1"/>
-<wire x1="64.77" y1="8.636" x2="67.31" y2="8.636" width="0" layer="19" extent="1-1"/>
-<wire x1="67.31" y1="6.096" x2="67.31" y2="8.636" width="0" layer="19" extent="1-1"/>
-<wire x1="64.77" y1="6.096" x2="64.77" y2="8.636" width="0" layer="19" extent="1-1"/>
-<wire x1="49.276" y1="17.272" x2="64.77" y2="8.636" width="0" layer="19" extent="1-1"/>
-<wire x1="44.45" y1="17.526" x2="49.276" y2="17.272" width="0" layer="19" extent="1-1"/>
-<wire x1="40.894" y1="17.272" x2="44.45" y2="17.526" width="0" layer="19" extent="1-1"/>
-<wire x1="37.60000625" y1="20.953503125" x2="40.894" y2="17.272" width="0" layer="19" extent="1-1"/>
-<wire x1="34.44328125" y1="20.395984375" x2="37.60000625" y2="20.953503125" width="0" layer="19" extent="1-1"/>
-<wire x1="32.766" y1="19.812" x2="34.44328125" y2="20.395984375" width="0" layer="19" extent="1-1"/>
-<wire x1="31.074271875" y1="19.38329375" x2="32.766" y2="19.812" width="0" layer="19" extent="1-1"/>
-<wire x1="23.495" y1="17.692" x2="31.074271875" y2="19.38329375" width="0" layer="19" extent="1-1"/>
-<wire x1="20.867" y1="13.335" x2="23.495" y2="17.692" width="0" layer="19" extent="1-1"/>
-<wire x1="13.161740625" y1="17.544196875" x2="20.867" y2="13.335" width="0" layer="19" extent="1-1"/>
-<wire x1="9.906" y1="14.732" x2="13.161740625" y2="17.544196875" width="0" layer="19" extent="1-1"/>
-<wire x1="9.652" y1="20.828" x2="13.161740625" y2="17.544196875" width="0" layer="19" extent="1-1"/>
-<wire x1="8.89" y1="27.94" x2="9.652" y2="20.828" width="0" layer="19" extent="1-1"/>
-<wire x1="10.68846875" y1="31.396496875" x2="8.89" y2="27.94" width="0" layer="19" extent="1-1"/>
-<wire x1="8.89" y1="36.068" x2="10.68846875" y2="31.396496875" width="0" layer="19" extent="1-1"/>
-<wire x1="16.256" y1="31.75" x2="10.68846875" y2="31.396496875" width="0" layer="19" extent="1-1"/>
-<wire x1="16.256" y1="35.052" x2="16.256" y2="31.75" width="0" layer="19" extent="1-1"/>
-<wire x1="17.526121875" y1="37.562028125" x2="16.256" y2="35.052" width="0" layer="19" extent="1-1"/>
-<wire x1="19.1864375" y1="38.119684375" x2="17.526121875" y2="37.562028125" width="0" layer="19" extent="1-16"/>
-<wire x1="22.86" y1="35.306" x2="19.1864375" y2="38.119684375" width="0" layer="19" extent="16-16"/>
-<wire x1="22.86" y1="32.004" x2="22.86" y2="35.306" width="0" layer="19" extent="1-1"/>
-<wire x1="26.6951625" y1="32.71620625" x2="22.86" y2="32.004" width="0" layer="19" extent="1-1"/>
-<wire x1="26.6951625" y1="37.28620625" x2="22.86" y2="35.306" width="0" layer="19" extent="1-1"/>
-<wire x1="26.416" y1="40.64" x2="26.6951625" y2="37.28620625" width="0" layer="19" extent="1-1"/>
-<wire x1="24.638" y1="40.64" x2="26.416" y2="40.64" width="0" layer="19" extent="1-1"/>
-<wire x1="25.467015625" y1="44.269509375" x2="24.638" y2="40.64" width="0" layer="19" extent="1-1"/>
 </signal>
 <signal name="+3.3V">
@@
 <wire x1="37.973" y1="29.050228125" x2="37.973" y2="31.623" width="0.381" layer="16"/>
 <via x="37.973" y="31.623" extent="1-16" drill="0.35"/>
-<wire x1="37.820278125" y1="45.32725" x2="39.090278125" y2="45.32725" width="0" layer="19" extent="1-1"/>
-<wire x1="36.550278125" y1="45.32725" x2="37.820278125" y2="45.32725" width="0" layer="19" extent="1-1"/>
-<wire x1="35.280278125" y1="45.32725" x2="36.550278125" y2="45.32725" width="0" layer="19" extent="1-1"/>
-<wire x1="45.542753125" y1="37.928903125" x2="39.090278125" y2="45.32725" width="0" layer="19" extent="1-1"/>
-<wire x1="37.973" y1="31.623" x2="45.542753125" y2="37.928903125" width="0" layer="19" extent="1-1"/>
-<wire x1="33.8751625" y1="35.00120625" x2="37.973" y2="31.623" width="0" layer="19" extent="1-1"/>
 </signal>
 <signal name="N$11">
@@
 <wire x1="12.346496875" y1="27.9727375" x2="12.4783125" y2="27.840921875" width="0.254" layer="1"/>
 <wire x1="12.38846875" y1="36.01046875" x2="12.38846875" y2="31.396496875" width="0.381" layer="1"/>
-<wire x1="14.590028125" y1="38.212028125" x2="12.38846875" y2="36.01046875" width="0.381" layer="1"/>
+<wire x1="12.38846875" y1="36.01046875" x2="14.590028125" y2="38.212028125" width="0.381" layer="1"/>
 <wire x1="12.4783125" y1="27.840921875" x2="20.042096875" y2="27.840921875" width="0.381" layer="1"/>
 <wire x1="20.042096875" y1="27.840921875" x2="20.137596875" y2="27.936421875" width="0.381" layer="1"/>
+<contactref element="U$1" pad="3"/>
+<wire x1="14.590028125" y1="38.212028125" x2="17.526121875" y2="38.212028125" width="0.381" layer="1"/>
 </signal>
 <signal name="ADJ">
@@
 </polygon>
 </signal>
-<signal name="N$1">
-<contactref element="U$1" pad="3"/>
-</signal>
 </signals>

Commit message: Reeeeeeeeeev 2 on the red line
Parts:
- removed +3.3V, 5V_3.3, GND3: (no value), SparkFun-Connectors:BANANA_CONN
- removed RSEN: 0.01, INA4181A4:CSS2H-2512
- added C6: 3300pF, SparkFun-Capacitors:0603
- added C7: 0.1uF, SparkFun-Capacitors:0603
- added C8, C9: 1.0uF, SparkFun-Capacitors:0603
- added CADJ1: 1000pF, SparkFun-Capacitors:0603
- added CBYP1: 1uF, SparkFun-Capacitors:0603
- added CIN1: 47uF, brick-capacitor-UCM1H331MNL1GS:CAPAE1030X1050N
- added COUT1: 100uF, PowerComponents:CTAN(7.30_4.30MM)
- added CVCC1: 0.47uF, SparkFun-Capacitors:0603
- added D5: SWITCHMODE_SCHOTTKY, Schottky Diode 8A - MBRD835LT4G:DPAK-3
- added J1, J2, J3, J4, J5: (no value), SparkFun-Connectors:1X01
- added J6, J7, J8, J9: (no value), Banana Plug PTH:BANANA_CONN_NO_THERM
- added JP1, JP2: JUMPER-SMT_2_NO_SILK, SparkFun-Jumpers:SMT-JUMPER_2_NO_SILK
- added L1: 15uH, Inductor_15uH - hcma1305:HCMA1305
- added Q2: (no value), SparkFun-DiscreteSemi:SO08
- added R2: 8.6k, SparkFun-Resistors:0603
- added R4: (no value), SparkFun-Resistors:0603
- added RADJ1: 1.8k, SparkFun-Resistors:0603
- added RFB3: 4.7k, SparkFun-Resistors:0603
- added RFB4: 15k, SparkFun-Resistors:0603
- added RT1: 82k, SparkFun-Resistors:0603
- added U$2: LM5085, Buck_Controller:LM5085
- added U$4: ADP7159ARDZ-04-R7, Linear Regulator - ADP7159:8-SOIC-EP
- C5: value 47uF -> 1.0uF
- R1: value 1.2 Ohms -> (none)
- moved D4 60.7 mm to (66.2, 48.5), turned to 0 degrees
- moved 1R 54.9 mm to (65.1, 46.2), turned to 270 degrees
- moved C4 43.1 mm to (61.7, 29.5), turned to 90 degrees
- moved C3 36.3 mm to (56.8, 33.1), turned to 0 degrees
- moved R1 34.5 mm to (68.8, 16.4), turned to 90 degrees
- moved Q1 30.7 mm to (15.4, 26.5), turned to 270 degrees
- moved CADJ 30.4 mm to (21.5, 14.5), flipped to the bottom, turned to 0 degrees
- moved U3 30.3 mm to (57.0, 27.4)
- moved RFB1 30.0 mm to (36.2, 14.3), turned to 270 degrees
- moved RADJ 29.5 mm to (21.4, 16.1), flipped to the bottom, turned to 0 degrees
- moved D3 29.2 mm to (61.3, 37.1)
- moved 3R 29.2 mm to (61.4, 33.9)
- moved RT 28.9 mm to (21.4, 12.9), flipped to the bottom, turned to 0 degrees
- moved CVCC 26.8 mm to (23.5, 18.0), flipped to the bottom, turned to 180 degrees
- moved C5 25.8 mm to (60.2, 18.2), flipped to the bottom
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Connections:
- net ADJ renamed ADJ2
- net FB renamed FB2
- net PGATE renamed PGATE2
- net RT renamed RT2
- net VCC renamed VCC2
- removed net +3.3V: +3.3V.P$1, 3R.2, C4.1, C5.1, U$3.4, U3.2, U3.4
- removed net +48V: 5R.2, CADJ.2, CBYP.1, CIN.+, CVCC.1, RADJ.2, RSEN.2, RT.2, U$1.8, U$3.1@1, U$3.1@2
- removed net +5V: 1R.2, 5V_3.3.P$1, C1.1, C3.1, COUT.+, L2.2, RFB2.1, U$3.3@1, U$3.3@2, U$3.3@3, U3.3
- removed net ISEN: Q1.1, Q1.2, Q1.3, RSEN.1, U$1.5
- removed net N$12: C5.2, R1.2
- removed net SWITCH: D1.4, L2.1, Q1.5, Q1.6, Q1.7, Q1.8, R3.1
- new net 18V: C6.1, CADJ.2, CBYP.1, CIN.+, CVCC.1, J2.1, L1.2, Q1.1, Q1.2, Q1.3, RADJ.2, RFB4.1, RT.2, U$1.8
- new net 3V3: 3R.2, C4.1, J4.1, J6.1, U$3.4, U$4.1, U$4.2, U3.2, U3.4
- new net 48V: 5R.2, CADJ1.2, CBYP1.1, CIN1.+, CVCC1.1, J1.1, J9.1, Q2.1, Q2.2, Q2.3, RADJ1.2, RT1.2, U$2.8, U$3.1@1, U$3.1@2
- new net 5V: 1R.2, C1.1, C3.1, COUT.+, COUT1.+, J3.1, J8.1, L2.2, RFB2.1, U$3.3@1, U$3.3@2, U$3.3@3, U$4.4, U$4.8, U3.3
- new net ADJ1: CADJ1.1, RADJ1.1, U$2.1
- new net BYP: C5.1, U$4.3
- new net FB1: C7.2, RFB3.1, RFB4.2, U$2.3
- new net ISEN1: JP1.2, U$2.5
- new net ISEN2: JP2.1, U$1.5
- new net N$1: C6.2, C7.1, R2.2
- new net PGATE1: Q2.4, U$2.6
- new net REF: C9.1, R1.2, U$4.6
- new net REF_SENSE: R1.1, R4.2, U$4.5
- new net RT1: RT1.1, U$2.2
- new net SWITCH1: D5.4, JP1.1, L1.1, Q2.5, Q2.6, Q2.7, Q2.8, R2.1
- new net SWITCH2: D1.4, JP2.2, L2.1, Q1.5, Q1.6, Q1.7, Q1.8, R3.1
- new net VCC1: CVCC1.2, U$2.7
- new net VREG: C8.1, U$4.7
- net GND: now also C5.2, C8.2, C9.2, CBYP1.2, CIN1.-, COUT1.-, D5.1, D5.3, J5.1, J7.1, R4.1, RFB3.2, U$2.4, U$4.PAD, U$4.PAD_BOT, U$4.PAD_VIA1, U$4.PAD_VIA2; no longer GND3.P$1, R1.1
Routing:
- net +3.3V: track 94.4 -> 0.00 mm, vias 1 -> 0
- net 3V3: track 0.00 -> 74.1 mm, vias 0 -> 5
- net 5V: track 0.00 -> 50.5 mm, vias 0 -> 2
- net +48V: track 44.3 -> 0.00 mm, vias 1 -> 0
- net 18V: track 0.00 -> 38.1 mm, vias 0 -> 2
- net SWITCH: track 28.6 -> 0.00 mm, vias 2 -> 0
- net ISEN: track 24.6 -> 0.00 mm
- net SWITCH2: track 0.00 -> 20.6 mm
- net 48V: track 0.00 -> 19.2 mm, vias 0 -> 2
- net PGATE1: track 0.00 -> 13.7 mm
- net FB1: track 0.00 -> 10.6 mm
- net +5V: track 9.24 -> 0.00 mm
- net FB2: track 22.0 -> 14.8 mm
- net N$11: track 10.3 -> 3.57 mm
- net GND: track 0.00 -> 5.96 mm, vias 20 -> 41
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- added copper zone on layer 1, net 18V
- added copper zone on layer 1, net 48V
- added copper zone on layer 1, net 5V
- added copper zone on layer 1, net SWITCH1
- added copper zone on layer 1, net SWITCH2
- added copper zone on layer 1, net X1
- added copper zone on layer 1, net X2
- removed copper zone on layer 1, net +48V
- removed copper zone on layer 1, net +5V
- removed copper zone on layer 1, net ADJ2
- removed copper zone on layer 1, net ISEN
- removed copper zone on layer 1, net SWITCH
- removed copper zone on layer 1, net X
Other:
- board text added: "48V - GND"
- board text added: "5V - 3V3 - GND - GND"
- board text added: "5V - GND"
- board text added: "ROV X13 Power Conversion v2 Bryce Sasser Read Hedl Grant Geyer 2/16/2021"
- board text removed: "ROV X13 Power Conversion v1 Bryce Sasser Read Hedl Grant Geyer 1/9/2021"
